Commit message: Add: RMUC sim env, Gmapping Add: License

File: src/sim_env/simulation/urdf/DJI2020AIROBOT/laser.xacro (robot description, xacro)
@@ -7,5 +7,5 @@
     <xacro:property name="laser_y" value="0.0" />
     <xacro:property name="laser_z" value="0.03" />
-    <!-- RPLIDAR -->
+    <!-- 2D LIDAR -->
     <link name="laser">
         <visual>
@@ -29,8 +29,8 @@
     </joint>
     <gazebo reference="laser">
-        <material>Gazebo/Black</material>
-        <sensor type="ray" name="rplidar">
+        <material>Gazebo/Green</material>
+        <sensor type="ray" name="laser">
             <pose>0 0 0 0 0 0</pose>
-            <visualize>true</visualize>
+            <visualize>false</visualize>
             <update_rate>5.5</update_rate>
             <ray>
@@ -39,5 +39,5 @@
                         <samples>360</samples>                        <!--旋转一周采的点数-->
                         <resolution>1</resolution>                        <!--每射线测距测距-->
-                        <min_angle>-3.14</min_angle>                        <!--采样范围，负逆顺正-->
+                        <min_angle>-3.14</min_angle>                        <!--采样范围，负逆正顺-->
                         <max_angle>3.14</max_angle>
                     </horizontal>
@@ -45,5 +45,5 @@
                 <range>
                     <min>0.10</min>                    <!--可检测距离  米-->
-                    <max>30.0</max>
+                    <max>12.0</max>
                     <resolution>0.01</resolution>
                 </range>
@@ -54,8 +54,12 @@
                 </noise>
             </ray>
-            <plugin name="gazebo_rplidar" filename="libgazebo_ros_ray_sensor.so">
-                <topicName>/scan</topicName>
-                <frameName>laser</frameName>
+            <plugin name="gazebo_laser" filename="libgazebo_ros_ray_sensor.so">
+                <topic>scan</topic>
+                <ros>
+                    <remapping>~/out:=scan</remapping>
+                </ros>
+                <output_type>sensor_msgs/LaserScan</output_type>
             </plugin>
+            <topic>scan</topic>
         </sensor>
     </gazebo>

File: src/sim_env/simulation/urdf/DJI2020AIROBOT/move.xacro (robot description, xacro)
@@ -53,23 +53,24 @@
     <gazebo>
         <plugin name="mecanum_controller" filename="libgazebo_ros_planar_move.so">
-            <updateRate>100.0</updateRate>
+            <ros>
+                <remapping>cmd_vel:=cmd_vel</remapping>
+                <remapping>odom:=odom</remapping>
+            </ros>
+            <update_rate>100.0</update_rate>
+            <publish_rate>100.0</publish_rate>
             <robotNamespace>/</robotNamespace>
-            <leftFrontJoint>left_wheel1base_link</leftFrontJoint>
-            <rightFrontJoint>right_wheel1base_link</rightFrontJoint>
-            <leftRearJoint>left_wheel2base_link</leftRearJoint>
-            <rightRearJoint>right_wheel2base_link</rightRearJoint>
+            <leftFrontJoint>front_left_wheel_joint</leftFrontJoint>
+            <rightFrontJoint>front_right_wheel_joint</rightFrontJoint>
+            <leftRearJoint>back_left_wheel_joint</leftRearJoint>
+            <rightRearJoint>back_right_wheel_joint</rightRearJoint>
             <wheelSeparation>0.48</wheelSeparation>
             <wheelDiameter>${wheel_radius * 2}</wheelDiameter>
-            <robotBaseFrame>base_link</robotBaseFrame>
             <torque>30</torque>
             <wheelAcceleration>1.8</wheelAcceleration>
-            <commandTopic>cmd_vel</commandTopic>
-            <odometryFrame>odom</odometryFrame>
-            <odometryTopic>odom</odometryTopic>
-            <odometryRate>20.000000</odometryRate>
-            <broadcastTF>1</broadcastTF>
             <covariance_x>0.000100</covariance_x>
             <covariance_y>0.000100</covariance_y>
             <covariance_yaw>0.000100</covariance_yaw>
+            <publish_odom>false</publish_odom>
+            <publish_odom_tf>false</publish_odom_tf>
         </plugin>
     </gazebo>

File: src/sim_env/simulation/urdf/SQUAREROBOT/Robot.xacro (robot description, xacro)
@@ -3,18 +3,22 @@
     <xacro:include filename="inertia.xacro" />
     <xacro:include filename="base.xacro" />
-    <xacro:include filename="support.xacro" />
     <xacro:include filename="wheel.xacro" />
     <xacro:include filename="move.xacro" />
     <xacro:include filename="camera.xacro" />
     <xacro:include filename="imu.xacro" />
-    <xacro:include filename="mid360.xacro" />
+    <xacro:include filename="laser.xacro" />
+    <xacro:include filename="$(find ros2_livox_simulation)/urdf/mid360.xacro" />
     <xacro:property name="PI" value="3.1415926535897931"/>
     <xacro:property name="package_name" value="simulation" />
-    <xacro:property name="wheel_offset_x" value="0.23" />
+    <xacro:property name="wheel_offset_x" value="0.21" />
     <xacro:property name="wheel_offset_y" value="0.29" />
-    <xacro:property name="wheel_offset_z" value="-0.02" />
+    <xacro:property name="wheel_offset_z" value="-0.09" />
+    <xacro:property name="laser_x" value="0.0" />
+    <xacro:property name="laser_y" value="0.0" />
+    <xacro:property name="laser_z" value="0.17" />
     <xacro:macro name="robot">
+        <!-- BASE_LINK -->
         <xacro:robot_base/>
-        <xacro:robot_support/>
+        <!-- WHEELS -->
         <xacro:omni_wheel prefix="front_right" parent="base_link" reflect="false">
             <origin xyz="${wheel_offset_x} -${wheel_offset_y} ${wheel_offset_z}" rpy="0 0 0"/>
@@ -29,7 +33,20 @@
             <origin xyz="-${wheel_offset_x} -${wheel_offset_y} ${wheel_offset_z}" rpy="0 0 0"/>
         </xacro:omni_wheel>
+        <!-- CAMERA -->
         <xacro:robot_camera/>
+        <!-- IMU -->
         <xacro:robot_imu/>
-        <xacro:robot_mid360/>
+        <!-- INVERTED LIVOX MID360 -->
+        <xacro:mid360 name="livox_frame" parent="base_link" topic="livox/lidar">
+            <origin xyz="0.0 0.0 0.53" rpy="${PI} 0 0"/>
+        </xacro:mid360>
+        <!-- NORMAL LIVOX MID360 -->
+        <!-- <xacro:mid360 name="livox_frame" parent="base_link" topic="livox/lidar">
+            <origin xyz="0.0 0.0 0.53" rpy="0 0 0"/>
+        </xacro:mid360> -->
+        <!-- 2D LIDAR -->
+        <!-- <xacro:robot_laser prefix="front" parent="base_link">
+            <origin xyz="${laser_x} ${laser_y} ${laser_z}" rpy="0 0 0"/>
+        </xacro:robot_laser> -->
     </xacro:macro>
     <xacro:robot/>

File: src/sim_env/simulation/urdf/SQUAREROBOT/base.xacro (robot description, xacro)
@@ -13,5 +13,5 @@
         <xacro:property name="base_link_hight" value="0.22" />
         <xacro:property name="earth_space" value="0" />
-        <xacro:property name="base_link_m" value="6.0" />
+        <xacro:property name="base_link_m" value="5.0" />
         <!-- BASE_FOOTPRINT -->
         <link name="base_footprint">
@@ -26,5 +26,5 @@
             <parent link="base_footprint" />
             <child link="base_link" />
-            <origin xyz="0 0 0.0" />
+            <origin xyz="0 0 0.09" />
         </joint>
         <gazebo reference="base_footprint">
@@ -38,5 +38,5 @@
                     <box size="${base_link_width} ${base_link_length} ${base_link_hight}"/>
                 </geometry>
-                <origin xyz="0 0 0.09" rpy="0 0 ${PI / 2}" />
+                <origin xyz="0 0 0" rpy="0 0 ${PI / 2}" />
                 <material name="black" />
             </visual>
@@ -55,5 +55,5 @@
             <visual>
                 <geometry>
-                    <box size="0.2 .28 .28"/>
+                    <box size="0.16 .16 .1"/>
                 </geometry>
                 <origin xyz="0 0 0" rpy="0 0 ${PI / 2}" />
@@ -64,13 +64,13 @@
             <collision>
                 <geometry>
-                    <box size="0.2 .28 .28"/>
+                    <box size="0.16 .16 .1"/>
                 </geometry>
             </collision>
-            <xacro:Box_inertial_matrix m="1.0" l="0.2" w="0.2" h="0.28" />
+            <xacro:Box_inertial_matrix m="0.2" l="0.16" w="0.16" h="0.1" />
         </link>
         <joint name="gimbal2baselink" type="fixed">
             <parent link="base_link"/>
             <child link="gimbal" />
-            <origin xyz="0 0 0.22001" rpy="0 0 0" />
+            <origin xyz="0 0 0.11" rpy="0 0 0" />
             <axis xyz="0 0 1" />
         </joint>

File: src/sim_env/simulation/urdf/SQUAREROBOT/camera.xacro (robot description, xacro)
@@ -6,7 +6,7 @@
         <xacro:property name="camera_height" value="0.025" />
         <xacro:property name="camera_mass" value="0.01" />
-        <xacro:property name="camera_x" value="0.125" />
+        <xacro:property name="camera_x" value="0.0" />
         <xacro:property name="camera_y" value="0.0" />
-        <xacro:property name="camera_z" value="0.15" />
+        <xacro:property name="camera_z" value="0.36" />
         <!-- CAMERA -->
         <link name="camera">
@@ -25,6 +25,6 @@
             <xacro:Box_inertial_matrix  m ="${camera_mass}" l ="${camera_length}" w ="${camera_width}" h ="${camera_height}" />
         </link>
-        <joint name="camera2gimbal" type="fixed">
-            <parent link="gimbal" />
+        <joint name="camera_joint" type="fixed">
+            <parent link="base_link" />
             <child link="camera" />
             <origin xyz="${camera_x} ${camera_y} ${camera_z}" />

File: src/sim_env/simulation/urdf/SQUAREROBOT/imu.xacro (robot description, xacro)
@@ -23,9 +23,9 @@
             </inertial>
         </link>
-        <joint name="imu2support" type="fixed">
-            <parent link="support_5"/>
+        <joint name="imu_joint" type="fixed">
+            <parent link="base_link"/>
             <child link="imu"/>
             <axis xyz="0 1 0" />
-            <origin xyz="0.0 0.0 -0.02" rpy="0 0 0"/>
+            <origin xyz="0.0 0.0 0.53" rpy="0 0 0"/>
         </joint>
         <gazebo reference="imu">
@@ -37,5 +37,5 @@
                 <visualize>true</visualize>
                 <topic>__default_topic__</topic>
-                <plugin filename="libgazebo_ros_imu_sensor.so" name="imu_plugin">
+                <plugin filename="libgazebo_ros_imu_sensor.so" name="gazebo_imu">
                     <topicName>imu</topicName>
                     <bodyName>imu_link</bodyName>

File: src/sim_env/simulation/urdf/SQUAREROBOT/move.xacro (robot description, xacro)
@@ -3,5 +3,4 @@
     <!-- JOINT_TRANS -->
     <xacro:macro name="joint_trans" params="joint_name">
-        <!-- Transmission is important to link the joints and the controller -->
         <transmission name="${joint_name}_trans">
             <type>transmission_interface/SimpleTransmission</type>
@@ -20,37 +19,33 @@
     <xacro:joint_trans joint_name="back_right_wheel_joint" />
     <gazebo reference="front_left_wheel_joint">
-        <mu1>0.5</mu1>
-        <mu2>0.5</mu2>
-        <kp>200000.0</kp>
-        <kd>10.0</kd>
-        <minDepth>0.001</minDepth>
-        <maxVel>1.0</maxVel>
+        <mu1 value="0.5"/>
+		<mu2 value="0.5"/>
+		<kp value="200000.0" />
+		<kd value="10.0" />
+		<fdir1 value="1 0 0"/>
         <turnGravityOff>false</turnGravityOff>
     </gazebo>
     <gazebo reference="front_right_wheel_joint">
-        <mu1>0.5</mu1>
-        <mu2>0.5</mu2>
-        <kp>200000.0</kp>
-        <kd>10.0</kd>
-        <minDepth>0.001</minDepth>
-        <maxVel>1.0</maxVel>
+        <mu1 value="0.5"/>
+		<mu2 value="0.5"/>
+		<kp value="200000.0" />
+		<kd value="10.0" />
+		<fdir1 value="1 0 0"/>
         <turnGravityOff>false</turnGravityOff>
     </gazebo>
     <gazebo reference="back_left_wheel_joint">
-        <mu1>0.5</mu1>
-        <mu2>0.5</mu2>
-        <kp>200000.0</kp>
-        <kd>10.0</kd>
-        <minDepth>0.001</minDepth>
-        <maxVel>1.0</maxVel>
+        <mu1 value="0.5"/>
+		<mu2 value="0.5"/>
+		<kp value="200000.0" />
+		<kd value="10.0" />
+		<fdir1 value="1 0 0"/>
         <turnGravityOff>false</turnGravityOff>
     </gazebo>
     <gazebo reference="back_right_wheel_joint">
-        <mu1>0.5</mu1>
-        <mu2>0.5</mu2>
-        <kp>200000.0</kp>
-        <kd>10.0</kd>
-        <minDepth>0.001</minDepth>
-        <maxVel>1.0</maxVel>
+        <mu1 value="0.5"/>
+		<mu2 value="0.5"/>
+		<kp value="200000.0" />
+		<kd value="10.0" />
+		<fdir1 value="1 0 0"/>
         <turnGravityOff>false</turnGravityOff>
     </gazebo>
@@ -58,5 +53,10 @@
     <gazebo>
         <plugin name="mecanum_controller" filename="libgazebo_ros_planar_move.so">
-            <updateRate>100.0</updateRate>
+            <ros>
+                <remapping>cmd_vel:=cmd_vel</remapping>
+                <remapping>odom:=odom</remapping>
+            </ros>
+            <update_rate>100.0</update_rate>
+            <publish_rate>100.0</publish_rate>
             <robotNamespace>/</robotNamespace>
             <leftFrontJoint>front_left_wheel_joint</leftFrontJoint>
@@ -66,15 +66,11 @@
             <wheelSeparation>0.56</wheelSeparation>
             <wheelDiameter>0.18</wheelDiameter>
-            <robotBaseFrame>base_link</robotBaseFrame>
             <torque>30</torque>
             <wheelAcceleration>1.8</wheelAcceleration>
-            <commandTopic>cmd_vel</commandTopic>
-            <odometryFrame>odom</odometryFrame>
-            <odometryTopic>odom</odometryTopic>
-            <odometryRate>20.000000</odometryRate>
-            <broadcastTF>1</broadcastTF>
             <covariance_x>0.000100</covariance_x>
             <covariance_y>0.000100</covariance_y>
             <covariance_yaw>0.000100</covariance_yaw>
+            <publish_odom>false</publish_odom>
+            <publish_odom_tf>false</publish_odom_tf>
         </plugin>
     </gazebo>

File: src/sim_env/simulation/urdf/SQUAREROBOT/support.xacro (robot description, xacro)
@@ -6,5 +6,5 @@
             <visual>
                 <geometry>
-                    <box size="0.01 0.02 0.36"/>
+                    <box size="0.01 0.02 0.42"/>
                 </geometry>
                 <origin xyz="0 0 0" rpy="0 0 ${PI / 2}" />
@@ -13,13 +13,13 @@
             <collision>
                 <geometry>
-                    <box size="0.01 0.02 0.36"/>
+                    <box size="0.01 0.02 0.42"/>
                 </geometry>
             </collision>
-            <xacro:Box_inertial_matrix m="0.1" l="0.01" w="0.02" h="0.36" />
+            <xacro:Box_inertial_matrix m="0.05" l="0.01" w="0.02" h="0.42" />
         </link>
         <joint name="1support2baselink" type="fixed">
             <parent link="base_link" />
             <child link="support_1" />
-            <origin xyz="0.0 0.24 0.3215" />
+            <origin xyz="0.0 0.24 0.2915" />
         </joint>
         <gazebo reference="support_1">
@@ -30,5 +30,5 @@
             <visual>
                 <geometry>
-                    <box size="0.01 0.02 0.36"/>
+                    <box size="0.01 0.02 0.42"/>
                 </geometry>
                 <origin xyz="0 0 0" rpy="0 0 ${PI / 2}" />
@@ -37,13 +37,13 @@
             <collision>
                 <geometry>
-                    <box size="0.01 0.02 0.36"/>
+                    <box size="0.01 0.02 0.42"/>
                 </geometry>
             </collision>
-            <xacro:Box_inertial_matrix m="0.1" l="0.01" w="0.02" h="0.36" />
+            <xacro:Box_inertial_matrix m="0.05" l="0.01" w="0.02" h="0.42" />
         </link>
         <joint name="2support2baselink" type="fixed">
             <parent link="base_link" />
             <child link="support_2" />
-            <origin xyz="0.0 -0.24 0.3215" />
+            <origin xyz="0.0 -0.24 0.2915" />
         </joint>
         <gazebo reference="support_2">
@@ -64,5 +64,5 @@
                 </geometry>
             </collision>
-            <xacro:Box_inertial_matrix m="0.1" l="0.01" w="0.02" h="0.18" />
+            <xacro:Box_inertial_matrix m="0.05" l="0.01" w="0.02" h="0.18" />
         </link>
         <joint name="3support2baselink" type="fixed">
@@ -88,5 +88,5 @@
                 </geometry>
             </collision>
-            <xacro:Box_inertial_matrix m="0.1" l="0.01" w="0.02" h="0.18" />
+            <xacro:Box_inertial_matrix m="0.05" l="0.01" w="0.02" h="0.18" />
         </link>
         <joint name="4support2baselink" type="fixed">
@@ -112,5 +112,5 @@
                 </geometry>
             </collision>
-            <xacro:Box_inertial_matrix m="0.1" l="0.18" w="0.18" h="0.02" />
+            <xacro:Box_inertial_matrix m="0.05" l="0.18" w="0.18" h="0.02" />
         </link>
         <joint name="5support2baselink" type="fixed">

File: src/sim_env/simulation/urdf/SQUAREROBOT/wheel.xacro (robot description, xacro)
@@ -1,38 +1,39 @@
-<robot name="wheel" xmlns:xacro="http://www.ros.org/wiki/xacro">
-  <xacro:property name="wheel_radius" value="0.09" />
-  <xacro:property name="wheel_height" value="0.0616" />
-  <xacro:property name="wheel_mass" value="0.5" />
-  <!-- WHEELS -->
-  <xacro:macro name="omni_wheel" params="prefix parent *origin reflect">
-    <joint name="${prefix}_wheel_joint" type="continuous">
-      <parent link="${parent}"/>
-      <child link="${prefix}_wheel_link"/>
-      <xacro:insert_block name="origin" />
-      <axis xyz="0 1 0" rpy="0 0 0" />
-      <limit effort="100" velocity="100"/>
-      <joint_properties damping="0.0" friction="0.0"/>
-    </joint>
-    <link name="${prefix}_wheel_link">
-      <visual>
-        <origin xyz="0 0 0" rpy="0 0 0" />
-        <xacro:if value="${reflect}">
-          <geometry>
-            <mesh filename="$(find ${package_name})/meshes/mecanum_wheel/mecanum_wheel_1.dae" />
-          </geometry>
-          </xacro:if>
-          <xacro:unless value="${reflect}">
-            <geometry>
-              <mesh filename="$(find ${package_name})/meshes/mecanum_wheel/mecanum_wheel_2.dae" />
-            </geometry>
-		    </xacro:unless>
-      </visual>
-      <collision>
-				<origin xyz="0 0 0" rpy="${PI/2} 0 0" />
-        <geometry>
-					<cylinder length="${wheel_height}" radius="${wheel_radius}" />
-        </geometry>
-      </collision>
-      <xacro:cylinder_inertial_matrix  m="${wheel_mass}" r="${wheel_radius}" h="${wheel_height}" />
-    </link>
-  </xacro:macro>
+<robot name="wheel"
+    xmlns:xacro="http://www.ros.org/wiki/xacro">
+    <xacro:property name="wheel_radius" value="0.09" />
+    <xacro:property name="wheel_height" value="0.0616" />
+    <xacro:property name="wheel_mass" value="0.05" />
+    <!-- WHEELS -->
+    <xacro:macro name="omni_wheel" params="prefix parent *origin reflect">
+        <joint name="${prefix}_wheel_joint" type="continuous">
+            <parent link="${parent}"/>
+            <child link="${prefix}_wheel_link"/>
+            <xacro:insert_block name="origin" />
+            <axis xyz="0 1 0" rpy="0 0 0" />
+            <limit effort="100" velocity="100"/>
+            <joint_properties damping="0.0" friction="0.0"/>
+        </joint>
+        <link name="${prefix}_wheel_link">
+            <visual>
+                <origin xyz="0 0 0" rpy="0 0 0" />
+                <xacro:if value="${reflect}">
+                    <geometry>
+                        <mesh filename="$(find ${package_name})/meshes/mecanum_wheel/mecanum_wheel_1.dae" />
+                    </geometry>
+                </xacro:if>
+                <xacro:unless value="${reflect}">
+                    <geometry>
+                        <mesh filename="$(find ${package_name})/meshes/mecanum_wheel/mecanum_wheel_2.dae" />
+                    </geometry>
+                </xacro:unless>
+            </visual>
+            <collision>
+                <origin xyz="0 0 0" rpy="${PI/2} 0 0" />
+                <geometry>
+                    <cylinder length="${wheel_height}" radius="${wheel_radius}" />
+                </geometry>
+            </collision>
+            <xacro:cylinder_inertial_matrix m="${wheel_mass}" r="${wheel_radius}" h="${wheel_height}" />
+        </link>
+    </xacro:macro>
 </robot>
